File: PCB/chrg/chrg.kicad_pcb (KiCad board)
At the start: 2 copper layers, 94.5 x 31 mm, 70 parts, among them U1 10k, U11 IP6518, U12 220uF, U13 IP6518, U14 220uF, U15 IP6518, U16 220uF, U17 IP6518, U18 220uF, U2 CH224K

Commit message: render
Parts:
- moved C53 0.21 mm to (84.2, 103.3)
- moved C38 0.21 mm to (44.5, 105.4)
- moved C43 0.21 mm to (45.3, 97.2)
- moved L7 0.21 mm to (36.8, 87.0)
- moved L8 0.21 mm to (57.8, 87.0)
- moved LED8 0.21 mm to (50.3, 105.2)
- moved R23 0.21 mm to (50.4, 102.5)
- moved U13 0.21 mm to (44.3, 100.8)
- moved USB10 0.21 mm to (36.3, 103.5)
- moved USB11 0.21 mm to (57.3, 103.5)
- moved LED7 0.21 mm to (29.3, 105.2)
- moved R20 0.21 mm to (29.4, 102.5)
- moved C37 0.21 mm to (43.9, 103.8)
- moved C39 0.21 mm to (42.2, 103.3)
- moved C40 0.21 mm to (40.9, 97.8)
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Routing:
- net /out1/VOUT1: track 35.2 -> 39.5 mm
- net /out2/VOUT1: track 35.2 -> 39.5 mm
- net /out3/VOUT1: track 35.2 -> 39.5 mm
- net /out2/CC1_1: track 15.7 -> 17.4 mm
- net /out3/CC1_1: track 15.7 -> 17.4 mm
- net /out1/CC1_1: track 15.7 -> 17.4 mm
- net /out1/CC2_1: track 11.8 -> 13.0 mm, vias 1 -> 2
- net /out2/CC2_1: track 11.8 -> 13.0 mm, vias 1 -> 2
- net /out3/CC2_1: track 11.8 -> 13.0 mm, vias 1 -> 2
Other:
- board text added: "chrg"

Commit message: should be correct now
Parts:
- moved C37 0.55 mm to (43.5, 103.4)
- moved C38 0.55 mm to (44.2, 105.0)
- moved C39 0.55 mm to (41.8, 102.9)
- moved C40 0.55 mm to (40.5, 97.4)
- moved C41 0.55 mm to (43.6, 96.9)
- moved C42 0.55 mm to (42.3, 96.9)
- moved C43 0.55 mm to (44.9, 96.8)
- moved C44 0.55 mm to (64.5, 103.4)
- moved C45 0.55 mm to (65.2, 105.0)
- moved C46 0.55 mm to (62.8, 102.9)
- moved C47 0.55 mm to (61.5, 97.4)
- moved C48 0.55 mm to (64.6, 96.9)
- moved C49 0.55 mm to (63.3, 96.9)
- moved C50 0.55 mm to (65.9, 96.8)
- moved C51 0.55 mm to (85.5, 103.4)
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Routing:
- net VIN: track 100.9 -> 128.3 mm
- net /out1/D1+: track 16.2 -> 23.2 mm
- net /out3/D1+: track 16.2 -> 23.2 mm
- net /out2/D1+: track 16.2 -> 23.2 mm
- net /out3/CC1_1: vias 1 -> 2
- net /out2/CC1_1: vias 1 -> 2
- net /out1/CC1_1: vias 1 -> 2
