File: PCB/chrg/chrg.kicad_pcb (KiCad board)
At the start: 2 copper layers, 94.5 x 31 mm, 70 parts, among them U1 10k, U11 IP6518, U12 220uF, U13 IP6518, U14 220uF, U15 IP6518, U16 220uF, U17 IP6518, U18 220uF, U2 CH224K

Commit message: e
Parts:
- removed C30, C35, C36, C37, C42, C43, C44, C49, C50, C51, C56, C57: 22uF, easyeda2kicad:C0402
- removed C31, C38, C45, C52: 100uF, easyeda2kicad:C0805
- removed R15, R18, R21, R24: 2Ω, easyeda2kicad:R0402
- added C10: 22uF, easyeda2kicad:C0603, F.Cu at (110.2, 93.2)
- added C11: 22uF, easyeda2kicad:C0603, F.Cu at (73.5, 49.2)
- added C12: 22uF, easyeda2kicad:C0603, F.Cu at (73.5, 59.2)
- added C13: 22uF, easyeda2kicad:C0603, F.Cu at (83.5, 49.2)
- added C14: 100uF, easyeda2kicad:C1206, F.Cu at (111.2, 83.1)
- added C2: 22uF, easyeda2kicad:C0603, F.Cu at (112.0, 106.5)
- added C3: 22uF, easyeda2kicad:C0603, F.Cu at (73.5, 43.8)
- added C4: 22uF, easyeda2kicad:C0603, F.Cu at (73.5, 53.8)
- added C5: 22uF, easyeda2kicad:C0603, F.Cu at (83.5, 43.8)
- added C6: 22uF, easyeda2kicad:C0603, F.Cu at (108.0, 105.2)
- added C7: 22uF, easyeda2kicad:C0603, F.Cu at (73.5, 46.5)
- added C8: 22uF, easyeda2kicad:C0603, F.Cu at (73.5, 56.5)
- added C9: 22uF, easyeda2kicad:C0603, F.Cu at (83.5, 46.5)
- added R3: 2Ω, easyeda2kicad:R0603, F.Cu at (103.8, 99.0)
- added R4: 2Ω, easyeda2kicad:R0603, F.Cu at (77.5, 43.7)
- added R5: 2Ω, easyeda2kicad:R0603, F.Cu at (77.5, 53.7)
- added R6: 2Ω, easyeda2kicad:R0603, F.Cu at (87.5, 43.7)
Routing:
- net GND: track 140.7 -> 134.5 mm, vias 47 -> 45
- net /out3/VOUT1: track 39.5 -> 38.1 mm
- net /out1/VOUT1: track 39.5 -> 38.1 mm
- net /out2/VOUT1: track 39.5 -> 38.1 mm
- net Net-(C54-Pad1): track 1.26 -> 0.00 mm
- net Net-(C47-Pad1): track 1.26 -> 0.00 mm
- net Net-(C40-Pad1): track 1.26 -> 0.00 mm
- net Net-(C53-Pad2): track 28.9 -> 28.1 mm
- net Net-(C46-Pad2): track 28.9 -> 28.1 mm
- net Net-(C39-Pad2): track 28.9 -> 28.1 mm
- net /out/VOUT1: track 39.5 -> 40.1 mm
Other:
- board size 94.5 x 31 mm -> 96.5 x 31 mm

Commit message: j
Parts:
- removed TP1, TP2: TestPoint, TestPoint:TestPoint_Pad_2.0x2.0mm
- moved R4 66.4 mm to (40.1, 98.6), turned to 180 degrees
- moved C7 65.2 mm to (44.3, 104.9), turned to 180 degrees
- moved C3 61.3 mm to (42.4, 96.7), turned to -90 degrees
- moved C9 58.4 mm to (86.3, 104.9), turned to 180 degrees
- moved R6 55.1 mm to (82.1, 98.6), turned to 180 degrees
- moved C5 52.8 mm to (84.4, 96.7), turned to -90 degrees
- moved C11 51.2 mm to (46.6, 92.8), turned to -90 degrees
- moved C8 49.0 mm to (65.3, 104.9), turned to 180 degrees
- moved R5 47.7 mm to (61.1, 98.6), turned to 180 degrees
- moved C4 44.0 mm to (63.4, 96.7), turned to -90 degrees
- moved C13 43.9 mm to (88.6, 92.8), turned to -90 degrees
- moved C12 34.1 mm to (67.6, 92.8), turned to -90 degrees
- moved C2 11.2 mm to (106.0, 97.0), turned to -90 degrees
- moved C14 3.91 mm to (112.5, 79.4), turned to 0 degrees
Routing:
- net GND: track 134.5 -> 150.1 mm, vias 45 -> 47
- net /out3/VOUT1: track 38.1 -> 40.1 mm
- net /out2/VOUT1: track 38.1 -> 40.1 mm
- net /out1/VOUT1: track 38.1 -> 40.1 mm
- net VIN: track 128.3 -> 126.4 mm, vias 40 -> 36
- net Net-(C54-Pad1): track 0.00 -> 1.52 mm
- net Net-(C47-Pad1): track 0.00 -> 1.52 mm
- net Net-(C40-Pad1): track 0.00 -> 1.52 mm
- net Net-(C53-Pad2): track 28.1 -> 28.9 mm
- net Net-(C46-Pad2): track 28.1 -> 28.9 mm
- net Net-(C39-Pad2): track 28.1 -> 28.9 mm

Commit message: yes
Parts:
- moved C3 0.83 mm to (41.9, 97.3), turned to -30 degrees
- moved C4 0.83 mm to (62.9, 97.3), turned to -30 degrees
- moved C5 0.83 mm to (83.9, 97.3), turned to -30 degrees
- moved C40 0.78 mm to (39.8, 97.8)
- moved C47 0.78 mm to (60.8, 97.8)
- moved C54 0.78 mm to (81.8, 97.8)
- moved C33 0.66 mm to (103.4, 97.8)
- moved C2 0.59 mm to (105.5, 97.3), turned to -30 degrees
- moved C41 0.40 mm to (43.6, 97.3)
- moved C48 0.40 mm to (64.6, 97.3)
- moved C55 0.40 mm to (85.6, 97.3)
- moved C11 0.40 mm to (46.6, 93.2)
- moved C12 0.40 mm to (67.6, 93.2)
- moved C13 0.40 mm to (88.6, 93.2)
- moved C39 0.40 mm to (41.8, 103.3)
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Routing:
- net VIN: track 126.4 -> 134.8 mm
- net GND: track 150.1 -> 155.1 mm

Commit message: delete 4x220uF 💀
Parts:
- removed U12, U14, U16, U18: 220uF, easyeda2kicad:C1206
Routing:
- net GND: track 155.1 -> 146.4 mm, vias 47 -> 43

Commit message: e
Parts:
- removed R2: 270Ω, lcsc:R0603
- added R21: 3.3kΩ, easyeda2kicad:R0402, F.Cu at (119.0, 104.5)
Routing:
- net /CFG2: track 9.30 -> 11.4 mm, vias 0 -> 2
