File: PCB/chrg/chrg.kicad_pcb (KiCad board)
At the start: 2 copper layers, 96.5 x 31 mm, 61 parts, among them U1 10k, U11 IP6518, U13 IP6518, U15 IP6518, U17 IP6518, U2 CH224K

Commit message: h
Parts:
- added H1: MountingHole, MountingHole:MountingHole_2.2mm_M2, F.Cu at (68.5, 82.0)
- added H2: MountingHole, MountingHole:MountingHole_2.2mm_M2, F.Cu at (29.0, 97.0)
- added H3: MountingHole, MountingHole:MountingHole_2.2mm_M2, F.Cu at (95.0, 97.0)
- added kobee-studio-6A88F8E8: Kobee Studio, kobee-studio-6A88F8A7, B.Cu at (47.3, 92.1)
