File: PCB/chrg/out.kicad_sch (KiCad schematic)
At the start: 15 parts, among them U11 IP6518, U12 220uF

Commit message: e
Parts:
- removed C30, C35, C36: 22uF, easyeda2kicad:C0402, symbol lcsc:CGA0402X5R226M6R3GT
- removed C31: 100uF, easyeda2kicad:C0805, symbol lcsc:JMK212BBJ107MG-TE
- removed R15: 2Ω, easyeda2kicad:R0402, symbol lcsc:FRC0402J2R0TS
- added C10, C2, C6: 22uF, easyeda2kicad:C0603, symbol lcsc:CL10A226MQ8NRNC
- added R3: 2Ω, easyeda2kicad:R0603, symbol lcsc:0603WAF200KT5E
- C32, C34: symbol lcsc:CC0402KRX7R9BB104 -> lcsc:CL05B104KO5NNNC; LCSC Part C131394 -> C1525; MPN CC0402KRX7R9BB104 -> CL05B104KO5NNNC; Manufacturer YAGEO(国巨) -> SAMSUNG(三星)
- C33: symbol lcsc:CL05B102KB5NNNC -> lcsc:0402B102K500NT; LCSC Part C14442 -> C1523; MPN CL05B102KB5NNNC -> 0402B102K500NT; Manufacturer SAMSUNG(三星) -> FH(风华)
- R16, R17: symbol lcsc:RC0402FR-073K3L -> lcsc:0402WGF3301TCE; LCSC Part C137992 -> C25890; MPN RC0402FR-073K3L -> 0402WGF3301TCE; Manufacturer YAGEO(国巨) -> UNI-ROYAL(厚声)
Connections:
- net GND: now also C10.1, C2.1, C6.2
- net VIN: now also C2.2, C6.1
- net VOUT1: now also C10.2
- net at C32.2, L6.1, U11.20 (LX)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: now also R3.1
- net at C33.1: now also R3.2

Commit message: delete 4x220uF 💀
Parts:
- removed U12: 220uF, easyeda2kicad:C1206, symbol lcsc:GRM31CR60G227ME11L
Changed lines of the file:
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@@
 	)
 	(junction
-		(at 106.68 36.83)
-		(diameter 0)
-		(color 0 0 0 0)
-	)
-	(junction
 		(at 62.23 54.61)
 		(diameter 0)
@@
 	(wire
 		(pts
-			(xy 95.25 36.83) (xy 106.68 36.83)
-		)
-		(stroke
-			(width 0)
-			(type default)
-		)
-	)
-	(wire
-		(pts
-			(xy 106.68 36.83) (xy 125.73 36.83)
+			(xy 95.25 36.83) (xy 125.73 36.83)
 		)
 		(stroke
@@
 	(symbol
 		(lib_id "power:GND")
-		(at 106.68 46.99 0)
-		(unit 1)
-		(body_style 1)
-		(exclude_from_sim no)
-		(in_bom yes)
-		(on_board yes)
-		(in_pos_files yes)
-		(dnp no)
-		(fields_autoplaced yes)
-		(property "Reference" "#PWR082"
-			(at 106.68 53.34 0)
-			(hide yes)
-			(show_name no)
-			(do_not_autoplace no)
-			(effects
-				(font
-					(size 1.27 1.27)
-				)
-			)
-		)
-		(property "Value" "GND"
-			(at 106.68 52.07 0)
-			(show_name no)
-			(do_not_autoplace no)
-			(effects
-				(font
-					(size 1.27 1.27)
-				)
-			)
-		)
-		(property "Footprint" ""
-			(at 106.68 46.99 0)
-			(hide yes)
-			(show_name no)
-			(do_not_autoplace no)
-			(effects
-				(font
-					(size 1.27 1.27)
-				)
-			)
-		)
-		(property "Datasheet" ""
-			(at 106.68 46.99 0)
-			(hide yes)
-			(show_name no)
-			(do_not_autoplace no)
-			(effects
-				(font
-					(size 1.27 1.27)
-				)
-			)
-		)
-		(property "Description" "Power symbol creates a global label with name \"GND\" , ground"
-			(at 106.68 46.99 0)
-			(hide yes)
-			(show_name no)
-			(do_not_autoplace no)
-			(effects
-				(font
-					(size 1.27 1.27)
-				)
-			)
-		)
-		(pin "1"
-		)
-		(instances
-			(project "chrg"
-				(path "/920d1772-7161-4a61-b520-2dcc7a0fc389/008349a9-e580-4854-bbec-06b61ef06a6b"
-					(reference "#PWR098")
-					(unit 1)
-				)
-				(path "/920d1772-7161-4a61-b520-2dcc7a0fc389/27617b1d-fd99-4571-a151-dc69e7cb18d7"
-					(reference "#PWR0130")
-					(unit 1)
-				)
-				(path "/920d1772-7161-4a61-b520-2dcc7a0fc389/530af39d-cd18-44af-97ca-e70c472550e3"
-					(reference "#PWR0114")
-					(unit 1)
-				)
-				(path "/920d1772-7161-4a61-b520-2dcc7a0fc389/f72d401b-64a9-418f-a9c0-87adba67f048"
-					(reference "#PWR082")
-					(unit 1)
-				)
-			)
-		)
-	)
-	(symbol
-		(lib_id "power:GND")
 		(at 114.3 71.12 180)
 		(unit 1)
@@
 					(unit 1)
 				)
-			)
-		)
-	)
-	(symbol
-		(lib_id "lcsc:GRM31CR60G227ME11L")
-		(at 106.68 41.91 90)
-		(unit 1)
-		(body_style 1)
-		(exclude_from_sim no)
-		(in_bom yes)
-		(on_board yes)
-		(in_pos_files yes)
-		(dnp no)
-		(fields_autoplaced yes)
-		(property "Reference" "U12"
-			(at 110.49 40.6399 90)
-			(show_name no)
-			(do_not_autoplace no)
-			(effects
-				(font
-					(size 1.27 1.27)
-				)
-				(justify right)
-			)
-		)
-		(property "Value" "220uF"
-			(at 110.49 43.1799 90)
-			(show_name no)
-			(do_not_autoplace no)
-			(effects
-				(font
-					(size 1.27 1.27)
-				)
-				(justify right)
-			)
-		)
-		(property "Footprint" "easyeda2kicad:C1206"
-			(at 114.3 41.91 0)
-			(hide yes)
-			(show_name no)
-			(do_not_autoplace no)
-			(effects
-				(font
-					(size 1.27 1.27)
-				)
-			)
-		)
-		(property "Datasheet" "https://www.lcsc.com/datasheet/C576503.pdf"
-			(at 116.84 41.91 0)
-			(hide yes)
-			(show_name no)
-			(do_not_autoplace no)
-			(effects
-				(font
-					(size 1.27 1.27)
-				)
-			)
-		)
-		(property "Description" ""
-			(at 106.68 41.91 0)
-			(hide yes)
-			(show_name no)
-			(do_not_autoplace no)
-			(effects
-				(font
-					(size 1.27 1.27)
-				)
-			)
-		)
-		(property "Manufacturer" "muRata(村田)"
-			(at 119.38 41.91 0)
-			(hide yes)
-			(show_name no)
-			(do_not_autoplace no)
-			(effects
-				(font
-					(size 1.27 1.27)
-				)
-			)
-		)
-		(property "MPN" "GRM31CR60G227ME11L"
-			(at 121.92 41.91 0)
-			(hide yes)
-			(show_name no)
-			(do_not_autoplace no)
-			(effects
-				(font
-					(size 1.27 1.27)
-				)
-			)
-		)
-		(property "LCSC Part" "C576503"
-			(at 124.46 41.91 0)
-			(hide yes)
-			(show_name no)
-			(do_not_autoplace no)
-			(effects
-				(font
-					(size 1.27 1.27)
-				)
-			)
-		)
-		(pin "2"
-		)
-		(pin "1"
-		)
-		(instances
-			(project "chrg"
-				(path "/920d1772-7161-4a61-b520-2dcc7a0fc389/008349a9-e580-4854-bbec-06b61ef06a6b"
-					(reference "U14")
-					(unit 1)
-				)
-				(path "/920d1772-7161-4a61-b520-2dcc7a0fc389/27617b1d-fd99-4571-a151-dc69e7cb18d7"
-					(reference "U18")
-					(unit 1)
-				)
-				(path "/920d1772-7161-4a61-b520-2dcc7a0fc389/530af39d-cd18-44af-97ca-e70c472550e3"
-					(reference "U16")
-					(unit 1)
-				)
-				(path "/920d1772-7161-4a61-b520-2dcc7a0fc389/f72d401b-64a9-418f-a9c0-87adba67f048"
-					(reference "U12")
-					(unit 1)
-				)

Commit message: bopt
Parts:
- removed L6: 22uH, easyeda2kicad:IND-SMD_L18.3-W18.2_MTF1810, symbol lcsc:MTF1810-220M
- added L1: SLO1350H220MTT, easyeda2kicad:IND-SMD_L14.4-W12.8, symbol lcsc:SLO1350H220MTT
Connections:
- net VOUT1: now also L1.2
- net at C32.2, R3.1, U11.20 (LX)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: now also L1.1
Changed lines of the file:
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@@
+	)
+	(symbol
+		(lib_id "lcsc:SLO1350H220MTT")
+		(at 69.85 36.83 0)
+		(unit 1)
+		(body_style 1)
+		(exclude_from_sim no)
+		(in_bom yes)
+		(on_board yes)
+		(in_pos_files yes)
+		(dnp no)
+		(fields_autoplaced yes)
+		(property "Reference" "L1"
+			(at 69.82 30.48 0)
+			(show_name no)
+			(do_not_autoplace no)
+			(effects
+				(font
+					(size 1.27 1.27)
+				)
+			)
+		)
+		(property "Value" "SLO1350H220MTT"
+			(at 69.82 33.02 0)
+			(show_name no)
+			(do_not_autoplace no)
+			(effects
+				(font
+					(size 1.27 1.27)
+				)
+			)
+		)
+		(property "Footprint" "easyeda2kicad:IND-SMD_L14.4-W12.8"
+			(at 69.85 44.45 0)
+			(hide yes)
+			(show_name no)
+			(do_not_autoplace no)
+			(effects
+				(font
+					(size 1.27 1.27)
+				)
+			)
+		)
+		(property "Datasheet" "https://lcsc.com/product-detail/Others_Sunltech-Tech-SLO1350H220MTT_C364085.html"
+			(at 69.85 46.99 0)
+			(hide yes)
+			(show_name no)
+			(do_not_autoplace no)
+			(effects
+				(font
+					(size 1.27 1.27)
+				)
+			)
+		)
+		(property "Description" ""
+			(at 69.85 36.83 0)
+			(hide yes)
+			(show_name no)
+			(do_not_autoplace no)
+			(effects
+				(font
+					(size 1.27 1.27)
+				)
+			)
+		)
+		(property "Manufacturer" "Sunltech(顺磁)"
+			(at 69.85 49.53 0)
+			(hide yes)
+			(show_name no)
+			(do_not_autoplace no)
+			(effects
+				(font
+					(size 1.27 1.27)
+				)
+			)
+		)
+		(property "MPN" "SLO1350H220MTT"
+			(at 69.85 52.07 0)
+			(hide yes)
+			(show_name no)
+			(do_not_autoplace no)
+			(effects
+				(font
+					(size 1.27 1.27)
+				)
+			)
+		)
+		(property "LCSC Part" "C364085"
+			(at 69.85 54.61 0)
+			(hide yes)
+			(show_name no)
+			(do_not_autoplace no)
+			(effects
+				(font
+					(size 1.27 1.27)
+				)
+			)
+		)
+		(pin "2"
+		)
+		(pin "1"
+		)
+		(instances
+			(project "chrg"
+				(path "/920d1772-7161-4a61-b520-2dcc7a0fc389/008349a9-e580-4854-bbec-06b61ef06a6b"
+					(reference "L2")
+					(unit 1)
+				)
+				(path "/920d1772-7161-4a61-b520-2dcc7a0fc389/27617b1d-fd99-4571-a151-dc69e7cb18d7"
+					(reference "L4")
+					(unit 1)
+				)
+				(path "/920d1772-7161-4a61-b520-2dcc7a0fc389/530af39d-cd18-44af-97ca-e70c472550e3"
+					(reference "L3")
+					(unit 1)
+				)
+				(path "/920d1772-7161-4a61-b520-2dcc7a0fc389/f72d401b-64a9-418f-a9c0-87adba67f048"
+					(reference "L1")
+					(unit 1)
+				)
+			)
+		)
 	)
 	(symbol
@@
 					(unit 1)
 				)
-			)
-		)
-	)
-	(symbol
-		(lib_id "lcsc:MTF1810-220M")
-		(at 69.85 36.83 0)
-		(unit 1)
-		(body_style 1)
-		(exclude_from_sim no)
-		(in_bom yes)
-		(on_board yes)
-		(in_pos_files yes)
-		(dnp no)
-		(fields_autoplaced yes)
-		(property "Reference" "L6"
-			(at 69.82 31.496 0)
-			(show_name no)
-			(do_not_autoplace no)
-			(effects
-				(font
-					(size 1.27 1.27)
-				)
-			)
-		)
-		(property "Value" "22uH"
-			(at 69.82 34.036 0)
-			(show_name no)
-			(do_not_autoplace no)
-			(effects
-				(font
-					(size 1.27 1.27)
-				)
-			)
-		)
-		(property "Footprint" "easyeda2kicad:IND-SMD_L18.3-W18.2_MTF1810"
-			(at 69.85 44.45 0)
-			(hide yes)
-			(show_name no)
-			(do_not_autoplace no)
-			(effects
-				(font
-					(size 1.27 1.27)
-				)
-			)
-		)
-		(property "Datasheet" "https://www.lcsc.com/datasheet/C5361009.pdf"
-			(at 69.85 46.99 0)
-			(hide yes)
-			(show_name no)
-			(do_not_autoplace no)
-			(effects
-				(font
-					(size 1.27 1.27)
-				)
-			)
-		)
-		(property "Description" ""
-			(at 69.85 36.83 0)
-			(hide yes)
-			(show_name no)
-			(do_not_autoplace no)
-			(effects
-				(font
-					(size 1.27 1.27)
-				)
-			)
-		)
-		(property "Manufacturer" "COILMX(迈翔科技)"
-			(at 69.85 49.53 0)
-			(hide yes)
-			(show_name no)
-			(do_not_autoplace no)
-			(effects
-				(font
-					(size 1.27 1.27)
-				)
-			)
-		)
-		(property "MPN" "MTF1810-220M"
-			(at 69.85 52.07 0)
-			(hide yes)
-			(show_name no)
-			(do_not_autoplace no)
-			(effects
-				(font
-					(size 1.27 1.27)
-				)
-			)
-		)
-		(property "LCSC Part" "C5361009"
-			(at 69.85 54.61 0)
-			(hide yes)
-			(show_name no)
-			(do_not_autoplace no)
-			(effects
-				(font
-					(size 1.27 1.27)
-				)
-			)
-		)
-		(pin "1"
-		)
-		(pin "2"
-		)
-		(instances
-			(project "chrg"
-				(path "/920d1772-7161-4a61-b520-2dcc7a0fc389/008349a9-e580-4854-bbec-06b61ef06a6b"
-					(reference "L7")
-					(unit 1)
-				)
-				(path "/920d1772-7161-4a61-b520-2dcc7a0fc389/27617b1d-fd99-4571-a151-dc69e7cb18d7"
-					(reference "L9")
-					(unit 1)
-				)
-				(path "/920d1772-7161-4a61-b520-2dcc7a0fc389/530af39d-cd18-44af-97ca-e70c472550e3"
-					(reference "L8")
-					(unit 1)
-				)
-				(path "/920d1772-7161-4a61-b520-2dcc7a0fc389/f72d401b-64a9-418f-a9c0-87adba67f048"
-					(reference "L6")
-					(unit 1)
-				)
